Commit message: Add camera to robot discription

File: franka_description/robots/common/franka_robot.xacro (robot description, xacro)
@@ -14,4 +14,8 @@
     <xacro:include filename="$(find franka_description)/robots/common/franka_arm.xacro" />
     <xacro:franka_arm arm_id="${arm_id}" safety_distance="0.03" gazebo="$(arg gazebo)" joint_limits="${joint_limits}"/>
+    <xacro:include filename="$(find realsense2_description)/urdf/_d435.urdf.xacro" /> <!-- URDF for d405 not available -->
+    <xacro:sensor_d435 parent="$(arg arm_id)_link8" name="fake_camera">
+      <origin xyz="0.04 -0.05 0.06" rpy="0.0 ${-pi/2} ${-pi/4}" />
+     </xacro:sensor_d435>
     <xacro:if value="$(arg hand)">
       <xacro:include filename="$(find franka_description)/robots/common/franka_hand.xacro"/>

Commit message: update approx location of camera

File: franka_description/robots/common/franka_robot.xacro (robot description, xacro)
@@ -16,5 +16,5 @@
     <xacro:include filename="$(find realsense2_description)/urdf/_d435.urdf.xacro" /> <!-- URDF for d405 not available -->
     <xacro:sensor_d435 parent="$(arg arm_id)_link8" name="fake_camera">
-      <origin xyz="0.04 -0.05 0.06" rpy="0.0 ${-pi/2} ${-pi/4}" />
+      <origin xyz="0.035 -0.05 0.06" rpy="0.0 ${-pi/2} ${-pi/4}" />
      </xacro:sensor_d435>
     <xacro:if value="$(arg hand)">
